File: hardware/eurorack_nvlp_1u/eurorack_nvlp_1u.kicad_pcb (KiCad board)
At the start: 2 copper layers, 50 x 39.6 mm, 36 parts, among them J101 GATE IN, J102 ENV_OUT, J103 POWER SUPPLY, Q101 MMBT3904, U101 STM32F030K6T6, U102 MCP4901-E/SN, U103 BU33SD5WG-TR

Commit message: small upgrades on the PCB
Parts:
- moved C110 0.20 mm to (44.6, 55.4)
- moved C111 0.20 mm to (54.6, 56.4)
- moved U102 0.20 mm to (49.6, 56.4)
Other:
- board text added: "+"
